Commit message: Updated joint limits

File: motoman_description/urdf/motoman.ros2_control.xacro (robot description, xacro)
@@ -8,6 +8,6 @@
       <joint name="joint_s">
           <command_interface name="position">
-          <param name="min">{-2*pi}</param>
-          <param name="max">{2*pi}</param>
+          <param name="min">{-pi}</param>
+          <param name="max">{pi}</param>
           </command_interface>
           <state_interface name="position">
@@ -16,6 +16,6 @@
       <joint name="joint_l">
           <command_interface name="position">
-          <param name="min">{-2*pi}</param>
-          <param name="max">{2*pi}</param>
+          <param name="min">{-1.9198}</param>
+          <param name="max">{1.9198}</param>
           </command_interface>
           <state_interface name="position">
@@ -23,4 +23,20 @@
       </joint>
       <joint name="joint_e">
+          <command_interface name="position">
+          <param name="min">{--2.9670}</param>
+          <param name="max">{-2.9670}</param>
+          </command_interface>
+          <state_interface name="position">
+          </state_interface>
+      </joint>
+      <joint name="joint_u">
+          <command_interface name="position">
+          <param name="min">{-2.2689}</param>
+          <param name="max">{2.2689}</param>
+          </command_interface>
+          <state_interface name="position">
+          </state_interface>
+      </joint>
+      <joint name="joint_r">
           <command_interface name="position">
           <param name="min">{-pi}</param>
@@ -30,24 +46,8 @@
           </state_interface>
       </joint>
-      <joint name="joint_u">
-          <command_interface name="position">
-          <param name="min">{-2*pi}</param>
-          <param name="max">{2*pi}</param>
-          </command_interface>
-          <state_interface name="position">
-          </state_interface>
-      </joint>
-      <joint name="joint_r">
-          <command_interface name="position">
-          <param name="min">{-2*pi}</param>
-          <param name="max">{2*pi}</param>
-          </command_interface>
-          <state_interface name="position">
-          </state_interface>
-      </joint>
       <joint name="joint_b">
           <command_interface name="position">
-          <param name="min">{-2*pi}</param>
-          <param name="max">{2*pi}</param>
+          <param name="min">{-1.9198}</param>
+          <param name="max">{1.9198}</param>
           </command_interface>
           <state_interface name="position">
@@ -56,6 +56,6 @@
       <joint name="joint_t">
           <command_interface name="position">
-          <param name="min">{-2*pi}</param>
-          <param name="max">{2*pi}</param>
+          <param name="min">{-pi}</param>
+          <param name="max">{pi}</param>
           </command_interface>
           <state_interface name="position">

Commit message: Added gripper as joint

File: motoman_description/urdf/motoman.ros2_control.xacro (robot description, xacro)
@@ -90,4 +90,10 @@
           </state_interface>
       </joint>
+      <joint name="motoman_gripper">
+          <command_interface name="position">
+          <param name="min">0</param>
+          <param name="max">1</param>
+          </command_interface>
+      </joint>
     </ros2_control>
   </xacro:macro>

File: motoman_description/urdf/motoman_sia20_macro.xacro (robot description, xacro)
@@ -201,5 +201,5 @@
 			<xacro:default_joint_misc/>
 		</joint>
-		<joint name = "motoman_link_t_to_gripper" type = "fixed">
+		<joint name = "motoman_gripper" type = "fixed">
 			<origin xyz = "0 0.02 0" rpy = "-1.57 0 0"/>
 			<parent link = "link_t"/>
