Commit message: RVIZ working

File: motoman_description/urdf/motoman.urdf.xacro (robot description, xacro)
@@ -6,5 +6,5 @@
     <xacro:include filename="$(find motoman_description)/urdf/motoman.ros2_control.xacro"/>
     <!-- Inclue gripper macro -->
-    <!-- <xacro:include filename="$(find aprs_description)/urdf/vacuum_gripper/vacuum_grippper_macro.xacro"/> -->
+    <xacro:include filename="$(find motoman_description)/urdf/gripper/motoman_gripper_macro.xacro"/>
     <link name="world"/>
     <!-- Run motoman macro -->
@@ -13,8 +13,7 @@
     <xacro:motoman_ros2_control name="motoman"/>
     <!-- Run gripper macro -->
-    <!-- <xacro:vacuum_gripper
-      parent="motoman_gripper_link"
-      prefix="motoman"
-      > -->
-    <!-- </xacro:vacuum_gripper> -->
+    <xacro:motoman_gripper
+      parent="link_t"
+      >
+    </xacro:motoman_gripper>
 </robot>

File: motoman_description/urdf/motoman_sia20_macro.xacro (robot description, xacro)
@@ -43,5 +43,5 @@
 			<child link = "motoman_base_link"/>
       	</joint>
-		<joint name="joint_r" type="revolute">
+		<joint name="joint_s" type="revolute">
 			<xacro:origin_joint_r/>
 			<parent link="motoman_base_link"/>
@@ -68,9 +68,9 @@
 		</link>
 		<!-- joint_e (link_s | joint_e) -->
-		<joint name="joint_e" type="revolute">
+		<joint name="joint_l" type="revolute">
 			<xacro:origin_joint_e/>
 			<parent link="link_s"/>
 			<child  link="link_l"/>
-			<axis xyz="0 0 1"/>
+			<axis xyz="0 0 -1"/>
 			<limit lower="-1.9198" upper="1.9198" effort="1000" velocity="2.2698"/>
 			<xacro:default_joint_misc/>
@@ -93,5 +93,5 @@
 		</link>
 		<!-- joint_l (link_l | joint_l) -->
-		<joint name="joint_l" type="revolute">
+		<joint name="joint_e" type="revolute">
 			<xacro:origin_joint_l/>
 			<parent link="link_l"/>
@@ -118,5 +118,5 @@
 		</link>
 		<!-- joint_t (link_e | joint_t) -->
-		<joint name="joint_t" type="revolute">
+		<joint name="joint_u" type="revolute">
 			<xacro:origin_joint_t/>
 			<parent link="link_e"/>
@@ -143,9 +143,9 @@
 		</link>
 		<!-- joint_u (link_u | joint_u) -->
-		<joint name="joint_u" type="revolute">
+		<joint name="joint_r" type="revolute">
 			<xacro:origin_joint_u/>
 			<parent link="link_u"/>
 			<child  link="link_r"/>
-			<axis xyz="0 1 0"/>
+			<axis xyz="0 -1 0"/>
 			<limit lower="-3.1415" upper="3.1415" effort="1000" velocity="3.4906"/>
 			<xacro:default_joint_misc/>
@@ -168,5 +168,5 @@
 		</link>
 		<!-- joint_s (link_r | joint_s) -->
-		<joint name="joint_s" type="revolute">
+		<joint name="joint_b" type="revolute">
 			<xacro:origin_joint_s/>
 			<parent link="link_r"/>
@@ -193,9 +193,9 @@
 		</link>
 		<!-- joint_b (link_b | joint_b) -->
-		<joint name="joint_b" type="revolute">
+		<joint name="joint_t" type="revolute">
 			<xacro:origin_joint_b/>
 			<parent link="link_b"/>
 			<child  link="link_t"/>
-			<axis xyz="0 1 0"/>
+			<axis xyz="0 -1 0"/>
 			<limit lower="-3.1415" upper="3.1415" effort="1000" velocity="7.0"/>
 			<xacro:default_joint_misc/>

Commit message: Updated with new base plate

File: motoman_description/urdf/motoman.urdf.xacro (robot description, xacro)
@@ -3,17 +3,30 @@
     <!-- Inclue motoman robot macro -->
     <xacro:include filename="$(find motoman_description)/urdf/motoman_sia20_macro.xacro"/>
+    <!-- Inclue gripper macro -->
+    <xacro:include filename="$(find motoman_description)/urdf/gripper/motoman_gripper_macro.xacro"/>
     <!-- Include ROS2 Control macro -->
     <xacro:include filename="$(find motoman_description)/urdf/motoman.ros2_control.xacro"/>
-    <!-- Inclue gripper macro -->
-    <xacro:include filename="$(find motoman_description)/urdf/gripper/motoman_gripper_macro.xacro"/>
     <link name="world"/>
+    <link name="motoman_base_plate">
+      <visual>
+        <origin rpy="0 0 0" xyz="0 0 0" />
+        <geometry>
+          <mesh filename="file://$(find motoman_description)/meshes/motoman_base_plate.stl" />
+        </geometry>
+        <material name="">
+            <color rgba="0.15 0.15 0.15 1.0" />
+        </material>
+      </visual>
+    </link>
+    <joint name = "motoman_base_plate_joint" type = "fixed">
+      <origin rpy = "0 0 0" xyz = "1.9685 0.1651 .0381"/>
+      <parent link = "world"/>
+      <child link = "motoman_base_plate"/>
+    </joint>
     <!-- Run motoman macro -->
-    <xacro:motoman_sia20d parent="world"/>
+    <xacro:motoman_sia20d parent="motoman_base_plate"/>
+    <!-- Run gripper macro -->
+    <xacro:motoman_gripper parent="link_t" />
     <!-- Run motoman macro -->
     <xacro:motoman_ros2_control name="motoman"/>
-    <!-- Run gripper macro -->
-    <xacro:motoman_gripper
-      parent="link_t"
-      >
-    </xacro:motoman_gripper>
 </robot>

Commit message: Updates to moveit and joint_trajectory_controller

File: motoman_description/urdf/motoman.urdf.xacro (robot description, xacro)
@@ -4,5 +4,5 @@
     <xacro:include filename="$(find motoman_description)/urdf/motoman_sia20_macro.xacro"/>
     <!-- Inclue gripper macro -->
-    <xacro:include filename="$(find motoman_description)/urdf/gripper/motoman_gripper_macro.xacro"/>
+    <xacro:include filename="$(find motoman_description)/urdf/motoman_gripper_macro.xacro"/>
     <!-- Include ROS2 Control macro -->
     <xacro:include filename="$(find motoman_description)/urdf/motoman.ros2_control.xacro"/>
@@ -20,5 +20,5 @@
     </link>
     <joint name = "motoman_base_plate_joint" type = "fixed">
-      <origin rpy = "0 0 0" xyz = "1.9685 0.1651 .0381"/>
+      <origin rpy = "0 0 3.14159" xyz = "1.9685 0.1651 .0381"/>
       <parent link = "world"/>
       <child link = "motoman_base_plate"/>

File: motoman_description/urdf/motoman_common.xacro (robot description, xacro)
@@ -8,5 +8,5 @@
 	<xacro:macro name="default_mesh" params="name">
 		<geometry>
-			<mesh filename="file://$(find motoman_description)/meshes/${name}.STL"/>
+			<mesh filename="file://$(find motoman_description)/meshes/${name}.stl"/>
 		</geometry>
 	</xacro:macro>

File: motoman_description/urdf/motoman_gripper_macro.xacro (robot description, xacro)
@@ -61,5 +61,5 @@
       <parent link="${parent}"/>
       <child link="motoman_gripper_link"/>
-      <origin xyz="0.2613 0 0" rpy="0 0 0"/>
+      <origin xyz="0 0.2588 0" rpy="-1.571 0 1.571"/>
     </joint>
     <!-- Finger 1 Joint -->

Commit message: testing fixes

File: motoman_description/urdf/motoman.urdf.xacro (robot description, xacro)
@@ -20,5 +20,5 @@
     </link>
     <joint name = "motoman_base_plate_joint" type = "fixed">
-      <origin rpy = "0 0 3.14159" xyz = "1.9685 0.1651 .0381"/>
+      <origin rpy = "0 0 3.14159" xyz = "1.9685 0.15 .0381"/>
       <parent link = "world"/>
       <child link = "motoman_base_plate"/>

Commit message: Alpha Release (#20)
* Driver Updates (#9)

* changed action namespace

* Motoman robot commander (untested)

* Lots of stuff - urdf changes and robot commander changes

* Updates (jtc not working 100%)

* Place in slot and pick from slot "working", visualization with planning scene started.

* Planning Scene Accurately reflects pick and place actions for large gear and large gear tray

* Movement

* Added new conveyor position for motoman moveit

* Added conveyor belt to the planning scene, the part itself needs slight design changes in addition to validating measurements for where the table starts

* Added code for adding attatched objects to planning scene

* Added conveyor to planning scene. Accuracy on conveyor needs to be improved. Pick and Place working.

* removed all instances of incorrect spelling of conveyor. With test Thursday to make sure all is working with robot commander

* should use time given by the trajectory

* Added ability to click points to determine corners and remove splotches for fanuc conveyor. To be moved to other locations, plus adding some labels.

* Much smother motion

* Updated file names and gripper macro

* Updated with new base plate

* Updates to moveit and joint_trajectory_controller

* Fixed motoman

* started building support for shared robot commander base class

* allow setting parameters from yaml file

* both robots working with shared base class

---------

Co-authored-by: jfernandez37 <jothomas0615@gmail.com>
Co-authored-by: rjs1442 <robert.seney@nist.gov>
Co-authored-by: Joseph Fernandez <joseph.fernandez@nist.gov>

* Vision system updates (#11)

* changed action namespace

* Lots of stuff - urdf changes and robot commander changes

* Place in slot and pick from slot "working", visualization with planning scene started.

* Planning Scene Accurately reflects pick and place actions for large gear and large gear tray

* Added conveyor belt to the planning scene, the part itself needs slight design changes in addition to validating measurements for where the table starts

* Added conveyor to planning scene. Accuracy on conveyor needs to be improved. Pick and Place working.

* removed all instances of incorrect spelling of conveyor. With test Thursday to make sure all is working with robot commander

* Added ability to click points to determine corners and remove splotches for fanuc conveyor. To be moved to other locations, plus adding some labels.

* Initial Commit for vision system. Working calibrate maps

* Added generate_grid_maps to vision_table. Fixed double waitkey issue. Added resets for any step that required it. Am able to calibrate on the fanuc table as well

* Updated calibration system. Fixed slider, changed rectangle drawing to use middle mouse button to avoid issues with zoom. Cleaned up classes to remove extra code and variables.

---------

Co-authored-by: rjs1442 <robert.seney@nist.gov>

* Vision updates (#12)

* Updated locate_trays_cb to work with fiducial marker and removed slot_pixel_publisher.

* Calibration updates

* made calibration tool into its own ros node. Started cleanup

* All user interface functions are coded

* Calibration is working

* refactored to work with new trays and calibration

* refactored stream handling into new class. Improved error recognition,

---------

Co-authored-by: rjs1442 <robert.seney@nist.gov>

* RVIZ config (#13)

* Integration Testing (#14)

* bug fix in sorting of holes. Added calibrations for motoman table and conveyor.

* calibrated fanuc_conveyor

* Small fixes

* added new meshes and fixed heights for trays and gears

* fixed s2l2 mesh

* Pick and place testing

* Pick and place testing

* added parameter from background value threshold

* testing fixes

* remove package

---------

Co-authored-by: rjs1442 <robert.seney@nist.gov>
Co-authored-by: Joseph Fernandez <joseph.fernandez@nist.gov>

* Vision Package Cleanup  (#15)

* Fixed linting errors and added docstrings

* linting and adding docstrings

* linting and docstrings

* added teach table calibration

* added parameters for other detection areas and added to launch

* PDDL Integration (#16)

* Add plansys2_msgs dependency and update service/action definitions

* Add ClearCurrentState service and implement execute plan action

* Refactor PDDL domain and problem definitions for dual robot kit building and handoff management

* Refactor PDDL domain and problem definitions for conveyor usage

* Update PDDL problem definition and refactor task planner for multi-robot tray management

* Refactor pick and place actions to support multiple robot clients for Fanuc and Motoman

* Fix pddl string

* Add RobotStatus message and remove GenerateInitState service

* Remove commented constants and unused predicates from PDDL domain and problem files

* Add RobotStatus subscriber and refactor task planner for operational state management

* Add MoveConveyorAction for conveyor control

* Refactor TaskPlanner to introduce process_trays method for tray processing and clean up goal string initialization

* Add conveyor_start_time member to MoveConveyorAction and replace sleep with time tracking for conveyor state management

* one pick and place for both robots concurrent execution

* updates

* testing

* added all nodes back to launch file

* removed imshow in detect trays

---------

Co-authored-by: Sanchit Kedia <sanchit.kedia@nist.gov>

* created akb application package and got live images working

* added reworked tray canvas

* changed tray canvas to use ros node

* Added service hanlders

* All custom widgets in one main window

* Added robot function frame

* added parameter to fix pddl

* Updates to pddl and interface

* Task planner changes

* reworked robot commander to handle changeover

* gui improvements

* robot changeover fixes

* fixes action progress

* Updates

* Added feature to tray canvas where robots pick and place gears which are clicked on the

* Ability to pick and place now dependent on whether gripper is open

* Added publishers for each of the controllers

* Added new controller status frame

* Copy paste issue

* Publishes true more often if on

* Fixed spacing on status page

* Pick and place working. Also controller status frame

* modified robot status frame

* Font fix

* new application

* added execute button back

* Added progress bar and plan rows change color depending on status

* Small fix

* Testing changes

* Should fix rows changing color in wrong order

* Plan frame working with only fanuc

* Change

* Demo working

* Fixed actual error in robot commander instead of GUI

* Needed

* Works

* Added select mode to pick/place

* Fixed place

* Open gripper sets held part to None

* Added control switch

* Select switch working

* Pick/place srv cbs check if gripper is open to pick

* Open gripper now allows you to pick another part successfully

* PDDL frame now works through keys instead of counting complete

* Fixes

* Added canvas tooltips and fixed type hinting

* Removed old code

* Small changes

* Final changes for demo

* Only updates image when it is selected

* Should be a more efficient status panel

* Cleaned op code and increased efficiency

* Fixed status panel

* Stopped the redrawing of the canvasases and will only update if it will be different

* Small bug fix

* Trying the service

* Lag issue much less of an issue

* Removed annoying log statement

* Drivers can handle e stops

* Updates to select mode

* Window holds it's size. Fixed seperator in status panel

* Status panel works on estop and error

---------

Co-authored-by: jfernandez37 <jothomas0615@gmail.com>
Co-authored-by: rjs1442 <robert.seney@nist.gov>
Co-authored-by: Joseph Fernandez <joseph.fernandez@nist.gov>
Co-authored-by: Sanchit Kedia <sanchit.kedia@nist.gov>

File: motoman_description/urdf/motoman.urdf.xacro (robot description, xacro)
@@ -3,17 +3,30 @@
     <!-- Inclue motoman robot macro -->
     <xacro:include filename="$(find motoman_description)/urdf/motoman_sia20_macro.xacro"/>
+    <!-- Inclue gripper macro -->
+    <xacro:include filename="$(find motoman_description)/urdf/motoman_gripper_macro.xacro"/>
     <!-- Include ROS2 Control macro -->
     <xacro:include filename="$(find motoman_description)/urdf/motoman.ros2_control.xacro"/>
-    <!-- Inclue gripper macro -->
-    <xacro:include filename="$(find motoman_description)/urdf/gripper/motoman_gripper_macro.xacro"/>
     <link name="world"/>
+    <link name="motoman_base_plate">
+      <visual>
+        <origin rpy="0 0 0" xyz="0 0 0" />
+        <geometry>
+          <mesh filename="file://$(find motoman_description)/meshes/motoman_base_plate.stl" />
+        </geometry>
+        <material name="">
+            <color rgba="0.15 0.15 0.15 1.0" />
+        </material>
+      </visual>
+    </link>
+    <joint name = "motoman_base_plate_joint" type = "fixed">
+      <origin rpy = "0 0 3.14159" xyz = "1.9685 0.15 .0381"/>
+      <parent link = "world"/>
+      <child link = "motoman_base_plate"/>
+    </joint>
     <!-- Run motoman macro -->
-    <xacro:motoman_sia20d parent="world"/>
+    <xacro:motoman_sia20d parent="motoman_base_plate"/>
+    <!-- Run gripper macro -->
+    <xacro:motoman_gripper parent="link_t" />
     <!-- Run motoman macro -->
     <xacro:motoman_ros2_control name="motoman"/>
-    <!-- Run gripper macro -->
-    <xacro:motoman_gripper
-      parent="link_t"
-      >
-    </xacro:motoman_gripper>
 </robot>
