Commit message: Fixed Fanuc controller lag

File: motoman_description/urdf/motoman_gripper_macro.xacro (robot description, xacro)
@@ -67,5 +67,5 @@
       <origin xyz="0.0 0.0 0.0" rpy="0.0 0.0 0.0" />
       <parent link="motoman_gripper_link" />
-      <child link="motoman_left_finger" />
+      <child link="motoman_left_finger" />is_estopped
       <axis xyz="0 -1 0" />
       <limit lower="0.0" upper="0.02" effort="1000" velocity="1000"/>
