Commit message: update part "Z" coordinates and add tool frame

File: fanuc_description/urdf/fanuc.ros2_control.xacro (robot description, xacro)
@@ -8,6 +8,6 @@
       <joint name="joint_1">
         <command_interface name="position">
-          <param name="min">{-2*pi}</param>
-          <param name="max">{2*pi}</param>
+          <param name="min">-2.967</param>
+          <param name="max">2.967</param>
         </command_interface>
         <state_interface name="position"/>
@@ -15,6 +15,6 @@
       <joint name="joint_2">
         <command_interface name="position">
-          <param name="min">{-2*pi}</param>
-          <param name="max">{2*pi}</param>
+          <param name="min">-1.745</param>
+          <param name="max">2.53</param>
         </command_interface>
         <state_interface name="position"/>
@@ -22,6 +22,6 @@
       <joint name="joint_3">
         <command_interface name="position">
-          <param name="min">{-2*pi}</param>
-          <param name="max">{2*pi}</param>
+          <param name="min">-2.447</param>
+          <param name="max">4.886</param>
         </command_interface>
         <state_interface name="position"/>
@@ -29,6 +29,6 @@
       <joint name="joint_4">
         <command_interface name="position">
-          <param name="min">{-2*pi}</param>
-          <param name="max">{2*pi}</param>
+          <param name="min">-3.316</param>
+          <param name="max">3.316</param>
         </command_interface>
         <state_interface name="position"/>
@@ -36,6 +36,6 @@
       <joint name="joint_5">
         <command_interface name="position">
-          <param name="min">{-2*pi}</param>
-          <param name="max">{2*pi}</param>
+          <param name="min">-2.18</param>
+          <param name="max">2.18</param>
         </command_interface>
         <state_interface name="position"/>

File: fanuc_description/urdf/fanuc_macro.xacro (robot description, xacro)
@@ -186,4 +186,15 @@
       </inertial>
     </link>
+    <link name="tool0">
+      <visual>
+        <origin rpy="0 1.571 0" xyz="-.085 0 0" />
+        <geometry>
+          <cylinder length="0.17" radius="0.04"/>
+        </geometry>
+        <material name="">
+          <color rgba="0.278431372549 0.278431372549 0.278431372549 1.0" />
+        </material>
+      </visual>
+    </link>
     <!-- joints -->
     <joint name = "base_joint_" type = "fixed">
@@ -234,4 +245,9 @@
         <limit effort="${joint6effort}" lower="${joint6lower}" upper="${joint6upper}" velocity="${joint6velocity}" />
     </joint>
+    <joint name="tool" type="fixed">
+        <origin xyz=".17 0 0" rpy="0 0 0"/>
+        <parent link="link_6"/>
+        <child link="tool0"/>
+    </joint>
   </xacro:macro>
 </robot>

Commit message: gripper controller test

File: fanuc_description/urdf/fanuc.ros2_control.xacro (robot description, xacro)
@@ -48,4 +48,20 @@
         <state_interface name="position"/>
       </joint>
+       <joint name="fanuc_prism1">
+          <command_interface name="position">
+          <param name="min">0</param>
+          <param name="max">0.02</param>
+          </command_interface>
+          <state_interface name="position">
+          </state_interface>
+      </joint>
+      <joint name="fanuc_prism2">
+          <command_interface name="position">
+          <param name="min">0</param>
+          <param name="max">0.02</param>
+          </command_interface>
+          <state_interface name="position">
+          </state_interface>
+      </joint>
     </ros2_control>
   </xacro:macro>

Commit message: added pnuematic gripper controller

File: fanuc_description/urdf/fanuc.ros2_control.xacro (robot description, xacro)
@@ -48,4 +48,12 @@
         <state_interface name="position"/>
       </joint>
+      <joint name="finger_1_joint">
+        <command_interface name="position"/>
+        <state_interface name="position"/>
+      </joint>
+      <joint name="finger_2_joint">
+        <command_interface name="position"/>
+        <state_interface name="position"/>
+      </joint>
     </ros2_control>
   </xacro:macro>

File: fanuc_description/urdf/fanuc.urdf.xacro (robot description, xacro)
@@ -3,4 +3,6 @@
   <!-- Inclue fanuc robot macro -->
   <xacro:include filename="$(find fanuc_description)/urdf/fanuc_macro.xacro"/>
+  <!-- Inclue gripper macro -->
+  <xacro:include filename="$(find fanuc_description)/urdf/fanuc_gripper_macro.xacro"/>
   <!-- Include ROS2 Control macro -->
   <xacro:include filename="$(find fanuc_description)/urdf/fanuc.ros2_control.xacro"/>
@@ -8,4 +10,6 @@
   <!-- Run fanuc macro -->
   <xacro:fanuc parent="world" />
+  <!-- Run gripper macro -->
+  <xacro:fanuc_gripper parent="link_6" />
   <!-- Run ros2 macro -->
   <xacro:fanuc_ros2_control name="fanuc" />

File: fanuc_description/urdf/fanuc_macro.xacro (robot description, xacro)
@@ -186,5 +186,5 @@
       </inertial>
     </link>
-    <link name="tool0">
+    <!-- <link name="tool0">
       <visual>
         <origin rpy="0 1.571 0" xyz="-.085 0 0" />
@@ -196,5 +196,5 @@
         </material>
       </visual>
-    </link>
+    </link> -->
     <!-- joints -->
     <joint name = "base_joint_" type = "fixed">
@@ -245,9 +245,9 @@
         <limit effort="${joint6effort}" lower="${joint6lower}" upper="${joint6upper}" velocity="${joint6velocity}" />
     </joint>
-    <joint name="tool" type="fixed">
+    <!-- <joint name="tool" type="fixed">
         <origin xyz=".17 0 0" rpy="0 0 0"/>
         <parent link="link_6"/>
         <child link="tool0"/>
-    </joint>
+    </joint> -->
   </xacro:macro>
 </robot>

Commit message: Lots of stuff - urdf changes and robot commander changes

File: fanuc_description/urdf/fanuc.ros2_control.xacro (robot description, xacro)
@@ -48,9 +48,9 @@
         <state_interface name="position"/>
       </joint>
-      <joint name="finger_1_joint">
+      <joint name="fanuc_left_finger_joint">
         <command_interface name="position"/>
         <state_interface name="position"/>
       </joint>
-      <joint name="finger_2_joint">
+      <joint name="fanuc_right_finger_joint">
         <command_interface name="position"/>
         <state_interface name="position"/>

File: fanuc_description/urdf/fanuc.urdf.xacro (robot description, xacro)
@@ -8,6 +8,28 @@
   <xacro:include filename="$(find fanuc_description)/urdf/fanuc.ros2_control.xacro"/>
   <link name="world"/>
+  <link name="fanuc_base_plate">
+    <visual>
+      <origin rpy="0 0 0" xyz="0 0 0" />
+      <geometry>
+        <mesh filename="file://$(find fanuc_description)/meshes/fanuc_base_plate.stl" />
+      </geometry>
+      <material name="">
+          <color rgba="0.15 0.15 0.15 1.0" />
+      </material>
+    </visual>
+    <collision>
+      <origin rpy="0 0 0" xyz="0 0 0" />
+      <geometry>
+        <mesh filename="file://$(find fanuc_description)/meshes/fanuc_base_plate.stl" />
+      </geometry>
+    </collision>
+  </link>
+  <joint name = "fanuc_base_plate_joint" type = "fixed">
+    <origin rpy = "0 0 0" xyz = "0.762 0.1778 .0254"/>
+    <parent link = "world"/>
+    <child link = "fanuc_base_plate"/>
+  </joint>
   <!-- Run fanuc macro -->
-  <xacro:fanuc parent="world" />
+  <xacro:fanuc parent="fanuc_base_plate" />
   <!-- Run gripper macro -->
   <xacro:fanuc_gripper parent="link_6" />

File: fanuc_description/urdf/fanuc_gripper_macro.xacro (robot description, xacro)
@@ -5,20 +5,26 @@
   ">
     <!-- Gripper Link -->
-    <link name="fanuc_gripper">
-      <visual name="fanuc_gripper_visual">
-        <origin rpy="0 1.571 0" xyz="-.085 0 0" />
+    <link name="fanuc_gripper_link">
+      <visual>
+        <origin rpy="0 0 0" xyz="0 0 0" />
         <geometry>
-          <cylinder length="0.17" radius="0.04"/>
+          <mesh filename="file://$(find fanuc_description)/meshes/gripper_link.stl"/>
         </geometry>
-        <material name="Cyan">
-          <color rgba="0 1.0 1.0 1.0"/>
-        </material>
+        <material name="">
+          <color rgba="0.15 0.15 0.15 1.0" />
+      </material>
       </visual>
+      <collision>
+        <origin rpy="0 0 0" xyz="0 0 0" />
+        <geometry>
+          <mesh filename="file://$(find fanuc_description)/meshes/gripper_link.stl" />
+        </geometry>
+      </collision>
     </link>
-     <link name="fanuc_finger_1">
+     <link name="fanuc_left_finger">
       <visual>
         <origin xyz="0 0 0" rpy="0 0 0" />
         <geometry>
-          <mesh filename="file://$(find fanuc_description)/meshes/visual/fanuc_finger_1.STL" />
+          <mesh filename="file://$(find fanuc_description)/meshes/fanuc_left_finger.stl" />
         </geometry>
         <material name="">
@@ -26,10 +32,16 @@
         </material>
       </visual>
+      <collision>
+        <origin rpy="0 0 0" xyz="0 0 0" />
+        <geometry>
+          <mesh filename="file://$(find fanuc_description)/meshes/fanuc_left_finger.stl" />
+        </geometry>
+      </collision>
     </link>
-    <link name="fanuc_finger_2">
+    <link name="fanuc_right_finger">
       <visual>
         <origin xyz="0 0 0" rpy="0 0 0" />
         <geometry>
-          <mesh filename="file://$(find fanuc_description)/meshes/visual/fanuc_finger_2.STL" />
+          <mesh filename="file://$(find fanuc_description)/meshes/fanuc_right_finger.stl" />
         </geometry>
         <material name="">
@@ -37,26 +49,38 @@
         </material>
       </visual>
+      <collision>
+        <origin rpy="0 0 0" xyz="0 0 0" />
+        <geometry>
+          <mesh filename="file://$(find fanuc_description)/meshes/fanuc_right_finger.stl" />
+        </geometry>
+      </collision>
     </link>
+    <link name="fanuc_tool0"/>
     <!-- Gripper Joint -->
-    <joint name="gripper_joint" type="fixed">
+    <joint name="fanuc_gripper_joint" type="fixed">
       <parent link="${parent}"/>
-      <child link="fanuc_gripper"/>
-      <origin xyz=".17 0 0" rpy="0 0 0"/>
+      <child link="fanuc_gripper_link"/>
+      <origin xyz="0.16046 0 0" rpy="0 0 0"/>
     </joint>
     <!-- Finger 1 Joint -->
-    <joint name="finger_1_joint" type="prismatic">
-      <origin xyz="0.0 0.02 0.010995" rpy="3.1416 6.123E-17 1.5708" />
-      <parent link="fanuc_gripper" />
-      <child link="fanuc_finger_1" />
-      <axis xyz="-1 0 0" />
+    <joint name="fanuc_left_finger_joint" type="prismatic">
+      <origin xyz="0.0 0.0 0.0" rpy="0.0 0.0 0.0" />
+      <parent link="fanuc_gripper_link" />
+      <child link="fanuc_left_finger" />
+      <axis xyz="0 -1 0" />
       <limit lower="0.0" upper="0.0075" effort="1000" velocity="1000"/>
     </joint>
     <!-- Finger 2 Joint -->
-    <joint name="finger_2_joint" type="prismatic">
-      <origin xyz="0.0 0 -0.010995" rpy="3.1416 -6.123E-17 -1.5708" />
-      <parent link="fanuc_gripper" />
-      <child link="fanuc_finger_2" />
-      <axis xyz="1 0 0" />
+    <joint name="fanuc_right_finger_joint" type="prismatic">
+      <origin xyz="0.0 0.0 0.0" rpy="0.0 0.0 0.0" />
+      <parent link="fanuc_gripper_link" />
+      <child link="fanuc_right_finger" />
+      <axis xyz="0 1 0" />
       <limit lower="0.0" upper="0.0075" effort="1000" velocity="1000"/>
+    </joint>
+    <joint name="fanuc_tool0_joint" type="fixed">
+      <origin xyz=" 0.042 0.0 0.0" rpy="0.0 1.57 0.0" />
+      <parent link="fanuc_gripper_link"/>
+      <child link="fanuc_tool0"/>
     </joint>
   </xacro:macro>

File: fanuc_description/urdf/fanuc_macro.xacro (robot description, xacro)
@@ -37,5 +37,5 @@
         <origin rpy="0 0 0" xyz="0 0 0" />
         <geometry>
-          <mesh filename="file://$(find fanuc_description)/meshes/visual/base_link.stl" />
+          <mesh filename="file://$(find fanuc_description)/meshes/base_link.stl" />
         </geometry>
         <material name="">
@@ -46,5 +46,5 @@
         <origin rpy="0 0 0" xyz="0 0 0" />
         <geometry>
-          <mesh filename="file://$(find fanuc_description)/meshes/collision/base_link.stl" />
+          <mesh filename="file://$(find fanuc_description)/meshes/base_link.stl" />
         </geometry>
       </collision>
@@ -58,14 +58,14 @@
         <origin rpy="0 0 0" xyz="0 0 0" />
         <geometry>
-          <mesh filename="file://$(find fanuc_description)/meshes/visual/link_1.stl" />
-        </geometry>
-        <material name="">
-          <color rgba="0.96 0.76 0.13 1.0" />
-        </material>
-      </visual>
-      <collision>
-        <origin rpy="0 0 0" xyz="0 0 0" />
-        <geometry>
-            <mesh filename="file://$(find fanuc_description)/meshes/collision/link_1.stl" />
+          <mesh filename="file://$(find fanuc_description)/meshes/link_1.stl" />
+        </geometry>
+        <material name="">
+          <color rgba="0.96 0.76 0.13 1.0" />
+        </material>
+      </visual>
+      <collision>
+        <origin rpy="0 0 0" xyz="0 0 0" />
+        <geometry>
+            <mesh filename="file://$(find fanuc_description)/meshes/link_1.stl" />
         </geometry>
       </collision>
@@ -80,14 +80,14 @@
         <origin rpy="0 0 0" xyz="0 0 0" />
         <geometry>
-          <mesh filename="file://$(find fanuc_description)/meshes/visual/link_2.stl" />
-        </geometry>
-        <material name="">
-          <color rgba="0.96 0.76 0.13 1.0" />
-        </material>
-      </visual>
-      <collision>
-        <origin rpy="0 0 0" xyz="0 0 0" />
-        <geometry>
-          <mesh filename="file://$(find fanuc_description)/meshes/collision/link_2.stl" />
+          <mesh filename="file://$(find fanuc_description)/meshes/link_2.stl" />
+        </geometry>
+        <material name="">
+          <color rgba="0.96 0.76 0.13 1.0" />
+        </material>
+      </visual>
+      <collision>
+        <origin rpy="0 0 0" xyz="0 0 0" />
+        <geometry>
+          <mesh filename="file://$(find fanuc_description)/meshes/link_2.stl" />
         </geometry>
       </collision>
@@ -102,5 +102,5 @@
           <origin rpy="0 0 0" xyz="0 0 0" />
           <geometry>
-              <mesh filename="file://$(find fanuc_description)/meshes/visual/link_3.stl" />
+              <mesh filename="file://$(find fanuc_description)/meshes/link_3.stl" />
           </geometry>
           <material name="">
@@ -111,5 +111,5 @@
           <origin rpy="0 0 0" xyz="0 0 0" />
           <geometry>
-              <mesh filename="file://$(find fanuc_description)/meshes/collision/link_3.stl" />
+              <mesh filename="file://$(find fanuc_description)/meshes/link_3.stl" />
           </geometry>
         </collision>
@@ -124,14 +124,14 @@
         <origin rpy="0 0 0" xyz="0 0 0" />
         <geometry>
-          <mesh filename="file://$(find fanuc_description)/meshes/visual/link_4.stl" />
-        </geometry>
-        <material name="">
-          <color rgba="0.96 0.76 0.13 1.0" />
-        </material>
-      </visual>
-      <collision>
-        <origin rpy="0 0 0" xyz="0 0 0" />
-        <geometry>
-          <mesh filename="file://$(find fanuc_description)/meshes/collision/link_4.stl" />
+          <mesh filename="file://$(find fanuc_description)/meshes/link_4.stl" />
+        </geometry>
+        <material name="">
+          <color rgba="0.96 0.76 0.13 1.0" />
+        </material>
+      </visual>
+      <collision>
+        <origin rpy="0 0 0" xyz="0 0 0" />
+        <geometry>
+          <mesh filename="file://$(find fanuc_description)/meshes/link_4.stl" />
         </geometry>
       </collision>
@@ -146,14 +146,14 @@
         <origin rpy="0 0 0" xyz="0 0 0" />
         <geometry>
-          <mesh filename="file://$(find fanuc_description)/meshes/visual/link_5.stl" />
-        </geometry>
-        <material name="">
-          <color rgba="0.96 0.76 0.13 1.0" />
-        </material>
-      </visual>
-      <collision>
-        <origin rpy="0 0 0" xyz="0 0 0" />
-        <geometry>
-            <mesh filename="file://$(find fanuc_description)/meshes/collision/link_5.stl" />
+          <mesh filename="file://$(find fanuc_description)/meshes/link_5.stl" />
+        </geometry>
+        <material name="">
+          <color rgba="0.96 0.76 0.13 1.0" />
+        </material>
+      </visual>
+      <collision>
+        <origin rpy="0 0 0" xyz="0 0 0" />
+        <geometry>
+            <mesh filename="file://$(find fanuc_description)/meshes/link_5.stl" />
         </geometry>
       </collision>
@@ -168,5 +168,5 @@
         <origin rpy="0 0 0" xyz="0 0 0" />
         <geometry>
-          <mesh filename="file://$(find fanuc_description)/meshes/visual/link_6.stl" />
+          <mesh filename="file://$(find fanuc_description)/meshes/link_6.stl" />
         </geometry>
         <material name="">
@@ -177,5 +177,5 @@
         <origin rpy="0 0 0" xyz="0 0 0" />
         <geometry>
-          <mesh filename="file://$(find fanuc_description)/meshes/collision/link_6.stl" />
+          <mesh filename="file://$(find fanuc_description)/meshes/link_6.stl" />
         </geometry>
       </collision>
@@ -198,5 +198,5 @@
     </link> -->
     <!-- joints -->
-    <joint name = "base_joint_" type = "fixed">
+    <joint name = "fanuc_base_joint" type = "fixed">
       <origin rpy = "0 0 0" xyz = "0 0 0"/>
       <parent link = "${parent}"/>
