Commit message: Place in slot and pick from slot "working", visualization with planning scene started.

File: fanuc_description/urdf/fanuc.urdf.xacro (robot description, xacro)
@@ -18,10 +18,4 @@
       </material>
     </visual>
-    <collision>
-      <origin rpy="0 0 0" xyz="0 0 0" />
-      <geometry>
-        <mesh filename="file://$(find fanuc_description)/meshes/fanuc_base_plate.stl" />
-      </geometry>
-    </collision>
   </link>
   <joint name = "fanuc_base_plate_joint" type = "fixed">

File: fanuc_description/urdf/fanuc_gripper_macro.xacro (robot description, xacro)
@@ -61,5 +61,5 @@
       <parent link="${parent}"/>
       <child link="fanuc_gripper_link"/>
-      <origin xyz="0.16046 0 0" rpy="0 0 0"/>
+      <origin xyz="0.152 0 0" rpy="0 0 0"/>
     </joint>
     <!-- Finger 1 Joint -->

Commit message: Driver Updates (#9)
* changed action namespace

* Motoman robot commander (untested)

* Lots of stuff - urdf changes and robot commander changes

* Updates (jtc not working 100%)

* Place in slot and pick from slot "working", visualization with planning scene started.

* Planning Scene Accurately reflects pick and place actions for large gear and large gear tray

* Movement

* Added new conveyor position for motoman moveit

* Added conveyor belt to the planning scene, the part itself needs slight design changes in addition to validating measurements for where the table starts

* Added code for adding attatched objects to planning scene

* Added conveyor to planning scene. Accuracy on conveyor needs to be improved. Pick and Place working.

* removed all instances of incorrect spelling of conveyor. With test Thursday to make sure all is working with robot commander

* should use time given by the trajectory

* Added ability to click points to determine corners and remove splotches for fanuc conveyor. To be moved to other locations, plus adding some labels.

* Much smother motion

* Updated file names and gripper macro

* Updated with new base plate

* Updates to moveit and joint_trajectory_controller

* Fixed motoman

* started building support for shared robot commander base class

* allow setting parameters from yaml file

* both robots working with shared base class

---------

Co-authored-by: jfernandez37 <jothomas0615@gmail.com>
Co-authored-by: rjs1442 <robert.seney@nist.gov>
Co-authored-by: Joseph Fernandez <joseph.fernandez@nist.gov>

File: fanuc_description/urdf/fanuc.urdf.xacro (robot description, xacro)
@@ -8,6 +8,22 @@
   <xacro:include filename="$(find fanuc_description)/urdf/fanuc.ros2_control.xacro"/>
   <link name="world"/>
+  <link name="fanuc_base_plate">
+    <visual>
+      <origin rpy="0 0 0" xyz="0 0 0" />
+      <geometry>
+        <mesh filename="file://$(find fanuc_description)/meshes/fanuc_base_plate.stl" />
+      </geometry>
+      <material name="">
+          <color rgba="0.15 0.15 0.15 1.0" />
+      </material>
+    </visual>
+  </link>
+  <joint name = "fanuc_base_plate_joint" type = "fixed">
+    <origin rpy = "0 0 0" xyz = "0.762 0.1778 .0254"/>
+    <parent link = "world"/>
+    <child link = "fanuc_base_plate"/>
+  </joint>
   <!-- Run fanuc macro -->
-  <xacro:fanuc parent="world" />
+  <xacro:fanuc parent="fanuc_base_plate" />
   <!-- Run gripper macro -->
   <xacro:fanuc_gripper parent="link_6" />

File: fanuc_description/urdf/fanuc_gripper_macro.xacro (robot description, xacro)
@@ -5,20 +5,26 @@
   ">
     <!-- Gripper Link -->
-    <link name="fanuc_gripper">
-      <visual name="fanuc_gripper_visual">
-        <origin rpy="0 1.571 0" xyz="-.085 0 0" />
+    <link name="fanuc_gripper_link">
+      <visual>
+        <origin rpy="0 0 0" xyz="0 0 0" />
         <geometry>
-          <cylinder length="0.17" radius="0.04"/>
+          <mesh filename="file://$(find fanuc_description)/meshes/gripper_link.stl"/>
         </geometry>
-        <material name="Cyan">
-          <color rgba="0 1.0 1.0 1.0"/>
-        </material>
+        <material name="">
+          <color rgba="0.15 0.15 0.15 1.0" />
+      </material>
       </visual>
+      <collision>
+        <origin rpy="0 0 0" xyz="0 0 0" />
+        <geometry>
+          <mesh filename="file://$(find fanuc_description)/meshes/gripper_link.stl" />
+        </geometry>
+      </collision>
     </link>
-     <link name="fanuc_finger_1">
+     <link name="fanuc_left_finger">
       <visual>
         <origin xyz="0 0 0" rpy="0 0 0" />
         <geometry>
-          <mesh filename="file://$(find fanuc_description)/meshes/visual/fanuc_finger_1.STL" />
+          <mesh filename="file://$(find fanuc_description)/meshes/fanuc_left_finger.stl" />
         </geometry>
         <material name="">
@@ -26,10 +32,16 @@
         </material>
       </visual>
+      <collision>
+        <origin rpy="0 0 0" xyz="0 0 0" />
+        <geometry>
+          <mesh filename="file://$(find fanuc_description)/meshes/fanuc_left_finger.stl" />
+        </geometry>
+      </collision>
     </link>
-    <link name="fanuc_finger_2">
+    <link name="fanuc_right_finger">
       <visual>
         <origin xyz="0 0 0" rpy="0 0 0" />
         <geometry>
-          <mesh filename="file://$(find fanuc_description)/meshes/visual/fanuc_finger_2.STL" />
+          <mesh filename="file://$(find fanuc_description)/meshes/fanuc_right_finger.stl" />
         </geometry>
         <material name="">
@@ -37,26 +49,38 @@
         </material>
       </visual>
+      <collision>
+        <origin rpy="0 0 0" xyz="0 0 0" />
+        <geometry>
+          <mesh filename="file://$(find fanuc_description)/meshes/fanuc_right_finger.stl" />
+        </geometry>
+      </collision>
     </link>
+    <link name="fanuc_tool0"/>
     <!-- Gripper Joint -->
-    <joint name="gripper_joint" type="fixed">
+    <joint name="fanuc_gripper_joint" type="fixed">
       <parent link="${parent}"/>
-      <child link="fanuc_gripper"/>
-      <origin xyz=".17 0 0" rpy="0 0 0"/>
+      <child link="fanuc_gripper_link"/>
+      <origin xyz="0.152 0 0" rpy="0 0 0"/>
     </joint>
     <!-- Finger 1 Joint -->
-    <joint name="finger_1_joint" type="prismatic">
-      <origin xyz="0.0 0.02 0.010995" rpy="3.1416 6.123E-17 1.5708" />
-      <parent link="fanuc_gripper" />
-      <child link="fanuc_finger_1" />
-      <axis xyz="-1 0 0" />
+    <joint name="fanuc_left_finger_joint" type="prismatic">
+      <origin xyz="0.0 0.0 0.0" rpy="0.0 0.0 0.0" />
+      <parent link="fanuc_gripper_link" />
+      <child link="fanuc_left_finger" />
+      <axis xyz="0 -1 0" />
       <limit lower="0.0" upper="0.0075" effort="1000" velocity="1000"/>
     </joint>
     <!-- Finger 2 Joint -->
-    <joint name="finger_2_joint" type="prismatic">
-      <origin xyz="0.0 0 -0.010995" rpy="3.1416 -6.123E-17 -1.5708" />
-      <parent link="fanuc_gripper" />
-      <child link="fanuc_finger_2" />
-      <axis xyz="1 0 0" />
+    <joint name="fanuc_right_finger_joint" type="prismatic">
+      <origin xyz="0.0 0.0 0.0" rpy="0.0 0.0 0.0" />
+      <parent link="fanuc_gripper_link" />
+      <child link="fanuc_right_finger" />
+      <axis xyz="0 1 0" />
       <limit lower="0.0" upper="0.0075" effort="1000" velocity="1000"/>
+    </joint>
+    <joint name="fanuc_tool0_joint" type="fixed">
+      <origin xyz=" 0.042 0.0 0.0" rpy="0.0 1.57 0.0" />
+      <parent link="fanuc_gripper_link"/>
+      <child link="fanuc_tool0"/>
     </joint>
   </xacro:macro>
