Commit message: Working in some capacity

File: motoman_description/urdf/gripper/motoman_gripper_macro.xacro (robot description, xacro)
@@ -6,15 +6,14 @@
         <!-- Gripper Link -->
         <link name="motoman_gripper_base">
-            <visual name="$motoman_gripper_base_visual">
+            <visual name="motoman_gripper_base_visual">
                 <origin xyz="0 0 0" rpy="0 0 0"/>
                 <geometry>
-                    <cylinder radius="0.05" length="0.05" />
+                    <mesh filename="file://$(find motoman_description)/meshes/motoman_gripper_link.STL" />
                 </geometry>
-                <material name="Grey"/>
             </visual>
-            <collision name="$motoman_gripper_base_collision">
+            <collision name="motoman_gripper_base_collision">
                 <origin xyz="0 0 -0.005" rpy="0 0 0"/>
                 <geometry>
-                <cylinder radius="0.05" length="0.05" />
+                    <mesh filename="file://$(find motoman_description)/meshes/motoman_gripper_link.STL" />
                 </geometry>
             </collision>
@@ -25,8 +24,8 @@
             </inertial>
         </link>
-        <joint name="$robot_to_gripper_base" type="fixed">
+        <joint name="robot_to_gripper_base" type="fixed">
             <parent link="${parent}"/>
             <child link="motoman_gripper_base"/>
-            <origin xyz="0.0 0.0 0.01" rpy="0.0 0.0 0.0"/>
+            <origin xyz="0.0 0.021 0.00" rpy="-1.57 -1.57 0.0"/>
         </joint>
         <link name="motoman_finger_1">
@@ -50,7 +49,5 @@
                 rpy="0 0 0" />
             <geometry>
-                <box>
-                    <size> 0.05 0.05 0.05 </size>
-                </box>
+                <mesh filename="file://$(find motoman_description)/meshes/motoman_finger_1.STL" />
             </geometry>
             <material
@@ -65,7 +62,5 @@
                 rpy="0 0 0" />
             <geometry>
-                <box>
-                    <size>0.05 0.05 0.05 </size>
-                </box>
+                <mesh filename="file://$(find motoman_description)/meshes/motoman_finger_1.STL" />
             </geometry>
             </collision>
@@ -75,5 +70,5 @@
             type="prismatic">
             <origin
-            xyz="0 0 0.1621"
+            xyz="0.0005 0 0.162"
             rpy="1.5708 0 0" />
             <parent
@@ -92,49 +87,45 @@
             name="motoman_finger_2">
             <inertial>
-            <origin
-                xyz="0.022998 0.021681 -9.8018E-06"
-                rpy="0 0 0" />
-            <mass
-                value="5" />
-            <inertia
-                ixx="1"
-                ixy="3.7227E-06"
-                ixz="1.199E-09"
-                iyy="1"
-                iyz="-5.7323E-09"
-                izz="1" />
+                <origin
+                    xyz="0.022998 0.021681 -9.8018E-06"
+                    rpy="0 0 0" />
+                <mass
+                    value="5" />
+                <inertia
+                    ixx="1"
+                    ixy="3.7227E-06"
+                    ixz="1.199E-09"
+                    iyy="1"
+                    iyz="-5.7323E-09"
+                    izz="1" />
             </inertial>
             <visual>
-            <origin
-                xyz="0 0 0"
-                rpy="0 0 0" />
-            <geometry>
-                <box>
-                    <size> 0.05 0.05 0.05 </size>
-                </box>
-            </geometry>
-            <material
-                name="">
-                <color
-                rgba="0.79216 0.81961 0.93333 1" />
-            </material>
+                <origin
+                    xyz="0 0 0"
+                    rpy="0 3.1415 0" />
+                <geometry>
+                    <mesh filename="file://$(find motoman_description)/meshes/motoman_finger_2.STL" />
+                </geometry>
+                <material
+                    name="">
+                    <color
+                    rgba="0.79216 0.81961 0.93333 1" />
+                </material>
             </visual>
             <collision>
-            <origin
-                xyz="0 0 0"
-                rpy="0 0 0" />
-            <geometry>
-                <box>
-                    <size> 0.05 0.05 0.05 </size>
-                </box>
-            </geometry>
+                <origin
+                    xyz="0 0 0"
+                    rpy="0 3.1415 0" />
+                <geometry>
+                    <mesh filename="file://$(find motoman_description)/meshes/motoman_finger_2.STL" />
+                </geometry>
             </collision>
         </link>
         <joint
-            name="motoman_prism_2"
+            name="motoman_prism2"
             type="prismatic">
             <origin
-            xyz="0 0 0.1621"
-            rpy="1.5708 0 3.1416" />
+            xyz="-0.0005 0 0.162"
+            rpy="1.5708 0 0" />
             <parent
             link="motoman_gripper_base" />
@@ -148,4 +139,5 @@
             effort="100"
             velocity="100" />
+            <!-- <mimic joint="motoman_prism_1" multiplier="1" offset="0"/> -->
         </joint>
     </xacro:macro>

File: motoman_description/urdf/motoman.ros2_control.xacro (robot description, xacro)
@@ -90,9 +90,19 @@
           </state_interface>
       </joint>
-      <joint name="motoman_gripper">
+      <joint name="motoman_prism1">
           <command_interface name="position">
           <param name="min">0</param>
-          <param name="max">1</param>
+          <param name="max">0.02</param>
           </command_interface>
+          <state_interface name="position">
+          </state_interface>
+      </joint>
+      <joint name="motoman_prism2">
+          <command_interface name="position">
+          <param name="min">0</param>
+          <param name="max">0.02</param>
+          </command_interface>
+          <state_interface name="position">
+          </state_interface>
       </joint>
     </ros2_control>

File: motoman_description/urdf/motoman_sia20_macro.xacro (robot description, xacro)
@@ -37,5 +37,4 @@
 			</collision>
 		</link>
-		<link name="motoman_gripper_link"/>
 		<joint name = "motoman_base_joint" type = "fixed">
 			<origin rpy = "0 0 0" xyz = "0 0 0"/>
@@ -201,9 +200,4 @@
 			<xacro:default_joint_misc/>
 		</joint>
-		<joint name = "motoman_gripper" type = "fixed">
-			<origin xyz = "0 0.02 0" rpy = "-1.57 0 0"/>
-			<parent link = "link_t"/>
-			<child link = "motoman_gripper_link"/>
-		</joint>
   </xacro:macro>
 </robot>

Commit message: Updates (jtc not working 100%)

File: motoman_description/urdf/gripper/motoman_gripper_macro.xacro (robot description, xacro)
@@ -5,6 +5,6 @@
         ">
         <!-- Gripper Link -->
-        <link name="motoman_gripper_base">
-            <visual name="motoman_gripper_base_visual">
+        <link name="motoman_gripper_link">
+            <visual>
                 <origin xyz="0 0 0" rpy="0 0 0"/>
                 <geometry>
@@ -12,5 +12,5 @@
                 </geometry>
             </visual>
-            <collision name="motoman_gripper_base_collision">
+            <collision>
                 <origin xyz="0 0 -0.005" rpy="0 0 0"/>
                 <geometry>
@@ -24,10 +24,10 @@
             </inertial>
         </link>
-        <joint name="robot_to_gripper_base" type="fixed">
+        <joint name="motoman_gripper_joint" type="fixed">
             <parent link="${parent}"/>
-            <child link="motoman_gripper_base"/>
+            <child link="motoman_gripper_link"/>
             <origin xyz="0.0 0.021 0.00" rpy="-1.57 -1.57 0.0"/>
         </joint>
-        <link name="motoman_finger_1">
+        <link name="motoman_left_finger">
             <inertial>
             <origin
@@ -49,5 +49,5 @@
                 rpy="0 0 0" />
             <geometry>
-                <mesh filename="file://$(find motoman_description)/meshes/motoman_finger_1.STL" />
+                <mesh filename="file://$(find motoman_description)/meshes/motoman_left_finger.STL" />
             </geometry>
             <material
@@ -62,10 +62,10 @@
                 rpy="0 0 0" />
             <geometry>
-                <mesh filename="file://$(find motoman_description)/meshes/motoman_finger_1.STL" />
+                <mesh filename="file://$(find motoman_description)/meshes/motoman_left_finger.STL" />
             </geometry>
             </collision>
         </link>
         <joint
-            name="finger_1_joint"
+            name="motoman_left_finger_joint"
             type="prismatic">
             <origin
@@ -73,7 +73,7 @@
             rpy="1.5708 0 0" />
             <parent
-            link="motoman_gripper_base" />
+            link="motoman_gripper_link" />
             <child
-            link="motoman_finger_1" />
+            link="motoman_left_finger" />
             <axis
             xyz="1 0 0" />
@@ -85,5 +85,5 @@
         </joint>
         <link
-            name="motoman_finger_2">
+            name="motoman_right_finger">
             <inertial>
                 <origin
@@ -105,5 +105,5 @@
                     rpy="0 3.1415 0" />
                 <geometry>
-                    <mesh filename="file://$(find motoman_description)/meshes/motoman_finger_2.STL" />
+                    <mesh filename="file://$(find motoman_description)/meshes/motoman_right_finger.STL" />
                 </geometry>
                 <material
@@ -118,10 +118,11 @@
                     rpy="0 3.1415 0" />
                 <geometry>
-                    <mesh filename="file://$(find motoman_description)/meshes/motoman_finger_2.STL" />
+                    <mesh filename="file://$(find motoman_description)/meshes/motoman_right_finger.STL" />
                 </geometry>
             </collision>
         </link>
+        <link name="motoman_tool0"/>
         <joint
-            name="finger_2_joint"
+            name="motoman_right_finger_joint"
             type="prismatic">
             <origin
@@ -129,7 +130,7 @@
             rpy="1.5708 0 0" />
             <parent
-            link="motoman_gripper_base" />
+            link="motoman_gripper_link" />
             <child
-            link="motoman_finger_2" />
+            link="motoman_right_finger" />
             <axis
             xyz="-1 0 0" />
@@ -141,4 +142,9 @@
             <!-- <mimic joint="motoman_prism_1" multiplier="1" offset="0"/> -->
         </joint>
+        <joint name="motoman_tool0_joint" type="fixed">
+            <origin xyz=" 0.042 0.0 0.0" rpy="0.0 1.57 0.0" />
+            <parent link="motoman_gripper_link"/>
+            <child link="motoman_tool0"/>
+        </joint>
     </xacro:macro>
 </robot>

File: motoman_description/urdf/motoman.ros2_control.xacro (robot description, xacro)
@@ -90,5 +90,5 @@
           </state_interface>
       </joint>
-      <joint name="finger_1_joint">
+      <joint name="motoman_left_finger_joint">
           <command_interface name="position">
             <param name="min">0</param>
@@ -98,5 +98,5 @@
           </state_interface>
       </joint>
-      <joint name="finger_2_joint">
+      <joint name="motoman_right_finger_joint">
           <command_interface name="position">
           <param name="min">0</param>
